File: power_supply/sps_power/sps_power.kicad_pcb (KiCad board)
At the start: 2 copper layers, 10 parts, among them U1 MC33063AD

Commit message: Interum commit
Parts:
- C1: footprint Capacitor_THT:CP_Radial_D6.3mm_P2.50mm -> Capacitor_THT:CP_Radial_D5.0mm_P2.50mm
- C2: footprint Capacitor_THT:CP_Radial_D5.0mm_P2.00mm -> Capacitor_SMD:C_1206_3216Metric_Pad1.42x1.75mm_HandSolder
- C3: value 470uF -> 220uF; footprint Capacitor_THT:CP_Radial_D12.5mm_P5.00mm -> Capacitor_SMD:CP_Elec_10x10
- TP1: value V-Out-Test-Point -> 5V_Out
- moved TP1 8.66 mm to (98.2, 68.6)
- moved D1 5.46 mm to (87.2, 89.7)
- moved L1 4.94 mm to (91.3, 77.7)
- moved C2 4.70 mm to (91.1, 89.5)
- moved R2 4.53 mm to (106.8, 88.5)
- moved C3 4.49 mm to (105.5, 75.7)
- moved C1 1.37 mm to (99.1, 93.7)
- moved R3 0.46 mm to (109.1, 88.4), turned to 90 degrees
Connections:
- net +12V renamed +24V

Commit message: Interum power supply cad commit
Parts:
- added J1: 5V Pwr, Connector_PinHeader_1.00mm:PinHeader_1x02_P1.00mm_Vertical, F.Cu at (103.5, 67.6)
Changed lines of the file:
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@@
     (tracks 0)
     (zones 0)
-    (modules 10)
+    (modules 11)
     (nets 8)
   )
@@
     (add_net "Net-(R2-Pad1)")
   )
+  (module Connector_PinHeader_1.00mm:PinHeader_1x02_P1.00mm_Vertical (layer F.Cu)
+    (at 103.505 67.564 180)
+    (descr "Through hole straight pin header, 1x02, 1.00mm pitch, single row")
+    (tags "Through hole pin header THT 1x02 1.00mm single row")
+    (fp_text reference J1 (at 0 -1.56) (layer F.SilkS)
+      (effects (font (size 1 1) (thickness 0.15)))
+    )
+    (fp_text value "5V Pwr" (at 0 2.56) (layer F.Fab)
+      (effects (font (size 1 1) (thickness 0.15)))
+    )
+    (fp_text user %R (at 0 0.5 90) (layer F.Fab)
+      (effects (font (size 0.76 0.76) (thickness 0.114)))
+    )
+    (fp_line (start 1.15 -1) (end -1.15 -1) (layer F.CrtYd) (width 0.05))
+    (fp_line (start 1.15 2) (end 1.15 -1) (layer F.CrtYd) (width 0.05))
+    (fp_line (start -1.15 2) (end 1.15 2) (layer F.CrtYd) (width 0.05))
+    (fp_line (start -1.15 -1) (end -1.15 2) (layer F.CrtYd) (width 0.05))
+    (fp_line (start -0.695 -0.685) (end 0 -0.685) (layer F.SilkS) (width 0.12))
+    (fp_line (start -0.695 0) (end -0.695 -0.685) (layer F.SilkS) (width 0.12))
+    (fp_line (start 0.608276 0.685) (end 0.695 0.685) (layer F.SilkS) (width 0.12))
+    (fp_line (start -0.695 0.685) (end -0.608276 0.685) (layer F.SilkS) (width 0.12))
+    (fp_line (start 0.695 0.685) (end 0.695 1.56) (layer F.SilkS) (width 0.12))
+    (fp_line (start -0.695 0.685) (end -0.695 1.56) (layer F.SilkS) (width 0.12))
+    (fp_line (start 0.394493 1.56) (end 0.695 1.56) (layer F.SilkS) (width 0.12))
+    (fp_line (start -0.695 1.56) (end -0.394493 1.56) (layer F.SilkS) (width 0.12))
+    (fp_line (start -0.635 -0.1825) (end -0.3175 -0.5) (layer F.Fab) (width 0.1))
+    (fp_line (start -0.635 1.5) (end -0.635 -0.1825) (layer F.Fab) (width 0.1))
+    (fp_line (start 0.635 1.5) (end -0.635 1.5) (layer F.Fab) (width 0.1))
+    (fp_line (start 0.635 -0.5) (end 0.635 1.5) (layer F.Fab) (width 0.1))
+    (fp_line (start -0.3175 -0.5) (end 0.635 -0.5) (layer F.Fab) (width 0.1))
+    (pad 2 thru_hole oval (at 0 1 180) (size 0.85 0.85) (drill 0.5) (layers *.Cu *.Mask)
+      (net 3 "Net-(C3-Pad1)"))
+    (pad 1 thru_hole rect (at 0 0 180) (size 0.85 0.85) (drill 0.5) (layers *.Cu *.Mask)
+      (net 1 GND))
+    (model ${KISYS3DMOD}/Connector_PinHeader_1.00mm.3dshapes/PinHeader_1x02_P1.00mm_Vertical.wrl
+      (at (xyz 0 0 0))
+      (scale (xyz 1 1 1))
+      (rotate (xyz 0 0 0))
+    )
+  )
   (module Capacitor_SMD:CP_Elec_10x10 (layer F.Cu)
