File: v1.0/signal-board/signal-board.sch (KiCad schematic (older format))
At the start: 35 parts, among them IC1 74HCT245, J1 Conn_02x09_Odd_Even, J2 Conn_02x08_Odd_Even, J3 5V Pwr Conn, J4 24V Screw Term, SW1 SW_MEC_5G, SW2 SW_MEC_5G, U1 ESP32-DEVKITC-32D, U2 MC33063AD

Commit message: v2 progress on schematic
Parts:
- removed C5: 100uF, Capacitor_SMD:C_Elec_6.3x7.7, symbol Device:CP1_Small
- removed C6: 470pF, Capacitor_SMD:C_1206_3216Metric_Pad1.42x1.75mm_HandSolder, symbol Device:CP1_Small
- removed C7: 220uF, Capacitor_SMD:CP_Elec_10x10, symbol Device:CP1_Small
- removed D2: 1N5819, Diode_SMD:D_SOD-123, symbol Device:D_Schottky
- removed J3: 5V Pwr Conn, Connector_PinHeader_2.54mm:PinHeader_1x02_P2.54mm_Vertical, symbol Connector:Conn_01x02_Male
- removed J4: 24V Screw Term, TerminalBlock_TE-Connectivity:TerminalBlock_TE_282834-2_1x02_P2.54mm_Horizontal, symbol Connector:Screw_Terminal_01x02
- removed L1: 220uH, Inductor_SMD:L_Bourns_SDR1806, symbol Device:L
- removed R14: 0.33 ohms, Resistor_SMD:R_0805_2012Metric_Pad1.15x1.40mm_HandSolder, symbol Device:R_Small_US
- removed R15: 1.2K, Resistor_SMD:R_0805_2012Metric_Pad1.15x1.40mm_HandSolder, symbol Device:R_Small_US
- removed R16: 3.6K, Resistor_SMD:R_0805_2012Metric_Pad1.15x1.40mm_HandSolder, symbol Device:R_Small_US
- removed U2: MC33063AD, Package_SO:SOIC-8_3.9x4.9mm_P1.27mm, symbol Regulator_Switching:MC33063AD
Connections:
- net labels removed: +24V, 5V_Out, 7V_to_24V_Input, Switching_Power_Supply
- wire segments 209 -> 168
