File: v1.1/signal-board/signal-board.sch (KiCad schematic (older format))
At the start: 44 parts, among them IC1 74HCT245, J1 Jack-DC, J2 Conn_01x12, J3 JST SM, J4 Conn_01x16, J5 switch_jumpers, J6 switch_jumpers, SW1 SW_MEC_5G, SW2 SW_MEC_5G, U1 TPS63060, U2 ESP32-DEVKITC-32D

Commit message: updated notes and updates from board review
Parts:
- added TP1: TestPoint, TestPoint:TestPoint_Pad_D1.0mm, symbol Connector:TestPoint
- C8: Supplier Digikey -> (none); Supplier Part 478-1395-1-ND -> (none)
- C9: Supplier Digikey -> (none); Supplier Part 08055C104KAT2A -> (none)
- R1: Supplier DigiKey -> (none)
- R4, R6: value 1k -> 1K; Supplier Digikey -> (none); Supplier Part 311-1.00KCRCT-ND -> (none)
Connections:
- net at R3.2, U1.5 (PG): now also TP1.1
Changed lines of the file:
@@
 Connection ~ 2300 7400
 Connection ~ 2300 7700
+Connection ~ 9900 9600
 NoConn ~ 7150 2800
 NoConn ~ 7150 2900
@@
 Wire Wire Line
 	9900 9600 8450 9600
+Wire Wire Line
+	9900 9600 10128 9600
 Wire Wire Line
 	10450 8600 10850 8600
@@
 3-12v
 $Comp
+L Connector:TestPoint TP1
+U 1 1 5F6FFFD0
+P 10128 9600
+F 0 "TP1" V 10083 9785 50  0000 L CNN
+F 1 "TestPoint" V 10173 9785 50  0000 L CNN
+F 2 "TestPoint:TestPoint_Pad_D1.0mm" H 10328 9600 50  0001 C CNN
+F 3 "~" H 10328 9600 50  0001 C CNN
+	1    10128 9600
+	0    1    1    0
+$EndComp
+$Comp
 L power:+3.3V #PWR0102
 U 1 1 5F4542FA
@@
 P 3025 1350
 F 0 "R4" V 3099 1374 50  0000 L CNN
-F 1 "1k" V 2951 1376 50  0000 L CNN
+F 1 "1K" V 2951 1376 50  0000 L CNN
 F 2 "Resistor_SMD:R_0402_1005Metric" H 3025 1350 50  0001 C CNN
 F 3 "~" H 3025 1350 50  0001 C CNN
-F 4 "Digikey" H 3025 1350 50  0001 C CNN "Supplier"
-F 5 "311-1.00KCRCT-ND" H 3025 1350 50  0001 C CNN "Supplier Part"
-F 6 "C11702" V 3025 1350 50  0001 C CNN "LCSC"
+F 4 "C11702" V 3025 1350 50  0001 C CNN "LCSC"
 	1    3025 1350
 	0    -1   -1   0
@@
 P 3025 2700
 F 0 "R6" V 3099 2724 50  0000 L CNN
-F 1 "1k" V 2951 2726 50  0000 L CNN
+F 1 "1K" V 2951 2726 50  0000 L CNN
 F 2 "Resistor_SMD:R_0402_1005Metric" H 3025 2700 50  0001 C CNN
 F 3 "~" H 3025 2700 50  0001 C CNN
-F 4 "Digikey" H 3025 2700 50  0001 C CNN "Supplier"
-F 5 "311-1.00KCRCT-ND" H 3025 2700 50  0001 C CNN "Supplier Part"
-F 6 "C11702" V 3025 2700 50  0001 C CNN "LCSC"
+F 4 "C11702" V 3025 2700 50  0001 C CNN "LCSC"
 	1    3025 2700
 	0    -1   -1   0
@@
 F 2 "Resistor_SMD:R_0402_1005Metric" V 9040 8740 50  0001 C CNN
 F 3 "~" H 9000 8750 50  0001 C CNN
-F 4 "DigiKey" H 9000 8750 50  0001 C CNN "Supplier"
-F 5 "" H 9000 8750 50  0001 C CNN "Price100"
-F 6 "C11702" H 9000 8750 50  0001 C CNN "LCSC"
+F 4 "" H 9000 8750 50  0001 C CNN "Price100"
+F 5 "C11702" H 9000 8750 50  0001 C CNN "LCSC"
 	1    9000 8750
 	1    0    0    -1
@@
 F 2 "Capacitor_SMD:C_0402_1005Metric" H 3275 1550 50  0001 C CNN
 F 3 "~" H 3275 1550 50  0001 C CNN
-F 4 "Digikey" H 3275 1550 50  0001 C CNN "Supplier"
-F 5 "478-1395-1-ND" H 3275 1550 50  0001 C CNN "Supplier Part"
-F 6 "C1525" H 3275 1550 50  0001 C CNN "LCSC"
+F 4 "C1525" H 3275 1550 50  0001 C CNN "LCSC"
 	1    3275 1550
 	1    0    0    -1
@@
 F 2 "Capacitor_SMD:C_0402_1005Metric" H 3275 2900 50  0001 C CNN
 F 3 "~" H 3275 2900 50  0001 C CNN
-F 4 "Digikey" H 3275 2900 50  0001 C CNN "Supplier"
-F 5 "08055C104KAT2A" H 3275 2900 50  0001 C CNN "Supplier Part"
-F 6 "C1525" H 3275 2900 50  0001 C CNN "LCSC"
+F 4 "C1525" H 3275 2900 50  0001 C CNN "LCSC"
 	1    3275 2900
 	1    0    0    -1
